Commit message: saving progress after locally: next to clean the code

File: depthai_descriptions/urdf/include/depthai_macro.urdf.xacro (robot description, xacro)
@@ -1,56 +1,95 @@
 <?xml version="1.0"?>
-<robot name="depthai_camera"
-    xmlns:xacro="http://ros.org/wiki/xacro">
-    <xacro:macro name="depthai_camera" params="camera_name camera_model parent base_frame
+<robot name="depthai_camera" xmlns:xacro="http://ros.org/wiki/xacro">
+<xacro:macro name="depthai_camera" params="camera_name camera_model parent base_frame
                                            cam_pos_x cam_pos_y cam_pos_z
-                                           cam_roll cam_pitch cam_yaw r:=0.8 g:=0.8 b:=0.8 a:=0.8 ">
-        <xacro:include filename="$(find depthai_descriptions)/urdf/include/base_macro.urdf.xacro"/>
-        <xacro:property name="M_PI" value="3.1415926535897931" />
-        <xacro:property name="model" value="${camera_model}" />
-        <xacro:property name="has_imu" value="false" />
-        <xacro:property name="baseline" value="0.075" />
-        <xacro:if value="${model == 'OAK-D'}">
-            <xacro:property name="has_imu" value="true" />
-        </xacro:if>
-        <xacro:base camera_name = "$(arg camera_name)" parent = "$(arg parent_frame)" camera_model = "$(arg camera_model)" base_frame = "$(arg base_frame)" cam_pos_x = "$(arg cam_pos_x)" cam_pos_y = "$(arg cam_pos_y)" cam_pos_z = "$(arg cam_pos_z)" cam_roll = "$(arg cam_roll)" cam_pitch = "$(arg cam_pitch)" cam_yaw = "$(arg cam_yaw)" has_imu="${has_imu}"/>
-        <!-- RGB Camera -->
-        <link name="${camera_name}_rgb_camera_frame" />
-        <joint name="${camera_name}_rgb_camera_joint" type="fixed">
+                                           cam_roll cam_pitch cam_yaw
+                                           r:=0.8 g:=0.8 b:=0.8 a:=0.8">
+    <xacro:property name="M_PI"     value="3.1415926535897931" />
+    <xacro:property name="model"    value="${camera_model}" />
+    <xacro:property name="has_imu" value="false" />
+    <!-- <xacro:if value="${model == 'BW1098OAK'}">
+    </xacro:if> -->
+    <xacro:property name="baseline" value="0.075" />
+    <xacro:if value="${model == 'OAK-D'}">
+      <xacro:property name="has_imu" value="true" />
+      <xacro:property name="imu_offset_x" value="0.0" />
+      <xacro:property name="imu_offset_y" value="-0.015" />
+      <xacro:property name="imu_offset_z" value="-0.013662" />
+      <xacro:property name="imu_r" value="0" />
+      <xacro:property name="imu_p" value="1.5708" />
+      <xacro:property name="imu_y" value="0" />
+    </xacro:if>
+    <!-- base_link of the sensor-->
+    <link name="${base_frame}"/>
+    <joint name="${camera_name}_center_joint" type="fixed">
+        <parent link="${parent}"/>
+        <child link="${base_frame}"/>
+        <origin xyz="${cam_pos_x} ${cam_pos_y} ${cam_pos_z}" rpy="${cam_roll} ${cam_pitch} ${cam_yaw}" />
+    </joint>
+<!-- device Center -->
+    <link name="${camera_name}_model_origin">
+        <visual>
+            <origin xyz="0 0 0" rpy="0 0 0"/>
+            <geometry>
+                <mesh filename="package://depthai_descriptions/urdf/models/${model}.stl" />
+            </geometry>
+            <material name="mat">
+                <color rgba="${r} ${g} ${b} ${a}"/>
+            </material>
+        </visual>
+    </link>
+    <joint name="${camera_name}_model_origin_joint" type="fixed">
+        <parent link="${base_frame}"/>
+        <child link="${camera_name}_model_origin"/>
+        <origin xyz="0 0 0" rpy="1.5708 0 1.5708" />
+    </joint>
+<!-- IMU -->
+    <xacro:if value="${has_imu}">
+        <link name="${camera_name}_imu_frame" />
+        <joint name="${camera_name}_imu_joint" type="fixed">
             <parent link="${base_frame}"/>
-            <child link="${camera_name}_rgb_camera_frame"/>
-            <origin xyz="0 0 0" rpy="0 0 0" />
+            <child link="${camera_name}_imu_frame"/>
+            <origin xyz="${imu_offset_x} ${imu_offset_y} ${imu_offset_z}" rpy="${imu_r} ${imu_p} ${imu_y}" />
         </joint>
-        <link name="${camera_name}_rgb_camera_optical_frame"/>
-        <joint name="${camera_name}_rgb_camera_optical_joint" type="fixed">
-            <origin xyz="0 0 0" rpy="-${M_PI/2} 0.0 -${M_PI/2}"/>
-            <parent link="${camera_name}_rgb_camera_frame"/>
-            <child link="${camera_name}_rgb_camera_optical_frame"/>
-        </joint>
-        <!-- Left Camera -->
-        <link name="${camera_name}_left_camera_frame" />
-        <joint name="${camera_name}_left_camera_joint" type="fixed">
-            <parent link="${base_frame}"/>
-            <child link="${camera_name}_left_camera_frame"/>
-            <origin xyz="0 ${baseline/2} 0" rpy="0 0 0" />
-        </joint>
-        <link name="${camera_name}_left_camera_optical_frame"/>
-        <joint name="${camera_name}_left_camera_optical_joint" type="fixed">
-            <origin xyz="0 0 0" rpy="-${M_PI/2} 0.0 -${M_PI/2}"/>
-            <parent link="${camera_name}_left_camera_frame"/>
-            <child link="${camera_name}_left_camera_optical_frame"/>
-        </joint>
-        <!-- right Camera -->
-        <link name="${camera_name}_right_camera_frame" />
-        <joint name="${camera_name}_right_camera_joint" type="fixed">
-            <parent link="${base_frame}"/>
-            <child link="${camera_name}_right_camera_frame"/>
-            <origin xyz="0 -${baseline/2} 0" rpy="0 0 0" />
-        </joint>
-        <link name="${camera_name}_right_camera_optical_frame"/>
-        <joint name="${camera_name}_right_camera_optical_joint" type="fixed">
-            <origin xyz="0 0 0" rpy="-${M_PI/2} 0.0 -${M_PI/2}"/>
-            <parent link="${camera_name}_right_camera_frame"/>
-            <child link="${camera_name}_right_camera_optical_frame"/>
-        </joint>
-    </xacro:macro>
+    </xacro:if>
+<!-- RGB Camera -->
+    <link name="${camera_name}_rgb_camera_frame" />
+    <joint name="${camera_name}_rgb_camera_joint" type="fixed">
+        <parent link="${base_frame}"/>
+        <child link="${camera_name}_rgb_camera_frame"/>
+        <origin xyz="0 0 0" rpy="0 0 0" />
+    </joint>
+    <link name="${camera_name}_rgb_camera_optical_frame"/>
+    <joint name="${camera_name}_rgb_camera_optical_joint" type="fixed">
+        <origin xyz="0 0 0" rpy="-${M_PI/2} 0.0 -${M_PI/2}"/>
+        <parent link="${camera_name}_rgb_camera_frame"/>
+        <child link="${camera_name}_rgb_camera_optical_frame"/>
+    </joint>
+<!-- Left Camera -->
+    <link name="${camera_name}_left_camera_frame" />
+    <joint name="${camera_name}_left_camera_joint" type="fixed">
+        <parent link="${base_frame}"/>
+        <child link="${camera_name}_left_camera_frame"/>
+        <origin xyz="0 ${baseline/2} 0" rpy="0 0 0" />
+    </joint>
+    <link name="${camera_name}_left_camera_optical_frame"/>
+    <joint name="${camera_name}_left_camera_optical_joint" type="fixed">
+        <origin xyz="0 0 0" rpy="-${M_PI/2} 0.0 -${M_PI/2}"/>
+        <parent link="${camera_name}_left_camera_frame"/>
+        <child link="${camera_name}_left_camera_optical_frame"/>
+    </joint>
+<!-- right Camera -->
+    <link name="${camera_name}_right_camera_frame" />
+    <joint name="${camera_name}_right_camera_joint" type="fixed">
+        <parent link="${base_frame}"/>
+        <child link="${camera_name}_right_camera_frame"/>
+        <origin xyz="0 -${baseline/2} 0" rpy="0 0 0" />
+    </joint>
+    <link name="${camera_name}_right_camera_optical_frame"/>
+    <joint name="${camera_name}_right_camera_optical_joint" type="fixed">
+        <origin xyz="0 0 0" rpy="-${M_PI/2} 0.0 -${M_PI/2}"/>
+        <parent link="${camera_name}_right_camera_frame"/>
+        <child link="${camera_name}_right_camera_optical_frame"/>
+    </joint>
+</xacro:macro>
 </robot>
